File: PCB/md_builtin_game_v2.2_no_TMSS_bypass.sch (EAGLE design)
At the start: 18 parts, among them IC1 MX29F1610A, IC2 ATF16V8BS

Commit message: Update PCB Version from v1.4 to v2.x - v2.1 has an optional (switchable) TMSS bypass mod included (TMSS bypass is enabled if /M30 (cart slot B30) is high and if the jumpers are set to on or to switchable with the pad ‚TS’ set to high) - v2.2 has no TMSS bypass mod included - v2.3 has the TMSS bypass mod included (TMSS bypass is enabled if /M30 (cart slot B30) is high) For all PCB versions, the PLD code v2.0 is to use.
Parts:
- removed C5: 100nF, arcadetv:C0805
- removed SJ3, SJ4: (no value), jumper:SJ
- removed U$2: /CS_K, arcadetv:PAD
- removed U$3: /CART_K, arcadetv:PAD
- removed U$4: /DISK (ExpPort B2), arcadetv:PAD
- removed U$5: BIG_Sel0, arcadetv:PAD
- removed U$7: BIG_Sel_1, arcadetv:PAD
- added /CART, /DISK, GS0, GS1: PAD, snes_div:PAD
- C1: value 22uF/6.3V -> 22uF; device rcl:CPOL-EUSMCB -> rcl:CPOL-EUSMCC
- C2: value 22uF -> 100nF; device rcl:CPOL-EUSMCB -> arcadetv:C0805
Connections:
- net /CHECK renamed CART_/CART
- removed net +5V: C1.+, C2.+, C3.2, C4.2, C5.2, IC1.!BYTE, IC1.!WE, IC1.VCC, IC2.VCC, U$6.A2, U$6.A31
- removed net ASIC_/CS: IC2.I4, U$2.P$1
- removed net CART_/CS: SJ4.2, U$6.B17
- removed net TMSS_MOD: IC2.OE, SJ3.1
- new net CART_/OE: IC2.I4, U$6.B17
- new net VCC: C1.+, C2.2, C3.2, C4.2, IC1.!BYTE, IC1.!WE, IC1.VCC, IC2.VCC, U$6.A2
- net /DISK: now also /DISK.P$1; no longer U$4.P$1
- net ASIC_/CART: now also /CART.P$1; no longer U$3.P$1
- net BIG_SEL0: now also GS0.P$1; no longer U$5.P$1
- net BIG_SEL1: now also GS1.P$1; no longer U$7.P$1
- net GND: now also C2.1, IC2.OE; no longer C2.-, C5.1, SJ3.2
- net N$1: no longer SJ4.1
Other:
- note added: "Cut the B32-line of the CartSlot! This will devide the signal /CART into: /CART_M -> towards CartSlot /CART_C -> towards IC4"
- note removed: "/CART_M -> towards CartSlot"
- note removed: "Add bypass-capacitors to all 3 ICs: 100nF Also a polarized cap (47uF) and a 22nF ceramic cap between +5V and GND on the supply-inputs."
- note removed: "Cut the B32-line of the CartSlot! This will devide the signal /CART into: /CART_M -> towards CartSlot /CART_K -> towards IC4"
- note removed: "TST2 same as /DISK???"
- moved on the sheet: C1, C3, C4
